Commit message: teleop con gamepad Logitech

File: description/lidar.xacro (robot description, xacro)
@@ -11,5 +11,5 @@
                 <cylinder radius="0.05" length="0.04"/>
             </geometry>
-            <material name="red"/>
+            <!-- <material name="red"/> -->
         </visual>
         <collision>
@@ -28,4 +28,5 @@
             <visualize>true</visualize>
             <update_rate>10</update_rate>
+            <always_on>true</always_on>
             <lidar>
                 <scan>
@@ -43,7 +44,11 @@
                 </range>
             </lidar>
-            <alwaysOn>true</alwaysOn>
-            <topic>scan</topic>
-            <frame_id>laser_frame_link</frame_id>
+            <plugin filename="libgazebo_ros_ray_sensor.so" name="laser_controller">
+                <ros>
+                    <remapping>~/out:=scan</remapping>
+                </ros>
+                <output_type>sensor_msgs/LaserScan</output_type>
+                <frame_name>laser_frame_link</frame_name>
+            </plugin>
         </sensor>
     </gazebo>
