Commit message: ajustes en el chasis y lidar

File: description/camera.xacro (robot description, xacro)
@@ -2,12 +2,12 @@
 <robot xmlns:xacro="http://www.ros.org/wiki/xacro" >
     <joint name="camera_joint" type="fixed">
-        <parent link="chassis_link"/>
+        <parent link="laser_base_link"/>
         <child link="camera_link"/>
-        <origin xyz="0.305 0 0.08" rpy="0 0 0"/>
+        <origin xyz="0.12 0 0.025" rpy="0 0 0"/>
     </joint>
     <link name="camera_link">
         <visual>
             <geometry>
-                <box size="0.010 0.03 0.03"/>
+                <box size="0.02 0.02 0.015"/>
             </geometry>
             <!-- <material name="red"/> -->
@@ -15,9 +15,16 @@
     </link>
     <joint name="camera_optical_joint" type="fixed">
-        <origin xyz="0 0 0" rpy="${-pi/2} 0 ${-pi/2}" />
+        <origin xyz="0.01 0 0" rpy="${-pi/2} 0 ${-pi/2}" />
         <parent link="camera_link" />
-        <child link="camera_link_optical" />
+        <child link="camera_optical_link" />
     </joint>
-    <link name="camera_link_optical"></link>
+    <link name="camera_optical_link">
+        <visual>
+            <geometry>
+                <cylinder radius="0.004" length="0.002"/>
+            </geometry>
+            <!-- <material name="red"/> -->
+        </visual>
+    </link>
     <gazebo reference="camera_link">
         <material>Gazebo/Red</material>

File: description/lidar.xacro (robot description, xacro)
@@ -1,13 +1,37 @@
 <?xml version="1.0"?>
 <robot xmlns:xacro="http://www.ros.org/wiki/xacro" >
+    <joint name="laser_base_joint" type="fixed">
+        <parent link="chassis_link"/>
+        <child link="laser_base_link"/>
+        <origin xyz="0.125 0 ${body_height}" rpy="0 0 0"/>
+    </joint>
+    <link name="laser_base_link">
+        <visual>
+            <origin xyz="0.025 0 0.02"/>
+            <geometry>
+                <box size="0.175 0.078 0.04"/>
+            </geometry>
+            <material name="white"/>
+        </visual>
+        <collision>
+            <origin xyz="0.025 0 0.02"/>
+            <geometry>
+                <box size="0.175 0.078 0.04"/>
+            </geometry>
+            <material name="white"/>
+        </collision>
+        <xacro:inertial_box mass="0.1" x="0.175" y="0.078" z="0.04">
+            <origin xyz="0 0 0" rpy="0 0 0"/>
+        </xacro:inertial_box>
+    </link>
     <joint name="laser_joint" type="fixed">
-        <parent link="chassis_link"/>
+        <parent link="laser_base_link"/>
         <child link="laser_frame_link"/>
-        <origin xyz="0.1 0 0.175" rpy="0 0 0"/>
+        <origin xyz="0.06 0 0.04" rpy="0 0 0"/>
     </joint>
     <link name="laser_frame_link">
         <visual>
             <geometry>
-                <cylinder radius="0.05" length="0.04"/>
+                <cylinder radius="0.03" length="0.04"/>
             </geometry>
             <!-- <material name="red"/> -->
@@ -15,11 +39,14 @@
         <collision>
             <geometry>
-                <cylinder radius="0.05" length="0.04"/>
+                <cylinder radius="0.03" length="0.04"/>
             </geometry>
         </collision>
-        <xacro:inertial_cylinder mass="0.1" length="0.04" radius="0.05">
+        <xacro:inertial_cylinder mass="0.1" length="0.04" radius="0.03">
             <origin xyz="0 0 0" rpy="0 0 0"/>
         </xacro:inertial_cylinder>
     </link>
+    <gazebo reference="laser_base_link">
+        <material>Gazebo/Black</material>
+    </gazebo>
     <gazebo reference="laser_frame_link">
         <material>Gazebo/Orange</material>

File: description/robot_core.xacro (robot description, xacro)
@@ -2,4 +2,26 @@
 <robot xmlns:xacro="http://www.ros.org/wiki/xacro" >
     <xacro:include filename="inertial_macros.xacro" />
+    <!-- ========== ROBOT PARAMETERS ========== -->
+    <!-- Chassis dimensions -->
+    <xacro:property name="body_length" value="0.345"/> <!-- chasis_largo -->
+    <xacro:property name="body_width" value="0.24"/> <!-- chasis_ancho -->
+    <xacro:property name="body_height" value="0.14"/> <!-- chasis_alto -->
+    <xacro:property name="body_mass" value="0.5"/> <!-- chasis_masa -->
+    <xacro:property name="body_x_offset" value="0.26"/> <!-- chasis_desplazamiento_x -->
+    <!-- Drive wheel properties -->
+    <xacro:property name="drive_wheel_radius" value="0.035"/> <!-- rueda_radio -->
+    <xacro:property name="drive_wheel_width" value="0.03"/> <!-- rueda_grosor -->
+    <xacro:property name="drive_wheel_mass" value="0.1"/> <!-- rueda_masa -->
+    <xacro:property name="wheel_base_width" value="0.14"/> <!-- rueda_separacion_y -->
+    <xacro:property name="wheel_mount_height" value="0.028"/> <!-- rueda_altura_z -->
+    <!-- Caster wheel properties -->
+    <xacro:property name="caster_radius" value="0.015"/> <!-- rueda_loca_radio -->
+    <xacro:property name="caster_mass" value="0.1"/> <!-- rueda_loca_masa -->
+    <xacro:property name="caster_x_pos" value="0.065"/> <!-- rueda_loca_posicion_x -->
+    <xacro:property name="caster_friction_coeff" value="0.001"/> <!-- rueda_loca_friccion -->
+    <!-- Calculated values -->
+    <xacro:property name="body_mid_x" value="${body_length/2}"/> <!-- chasis_centro_x -->
+    <xacro:property name="body_mid_z" value="${body_height/2}"/> <!-- chasis_centro_z -->
+    <!-- ========== MATERIALS ========== -->
     <material name="white">
         <color rgba="1 1 1 1" />
@@ -14,4 +36,5 @@
         <color rgba="0 0 0 1" />
     </material>
+    <!-- ========== LINKS AND JOINTS ========== -->
     <!-- BASE LINK-->
     <link name="base_link">
@@ -21,23 +44,23 @@
         <parent link="base_link" />
         <child link="chassis_link" />
-        <origin xyz="-0.1 0 0"/>
+        <origin xyz="-${body_x_offset} 0 0"/>
     </joint>
     <link name="chassis_link">
         <visual>
-            <origin xyz="0.15 0 0.075"/>
+            <origin xyz="${body_mid_x} 0 ${body_mid_z}"/>
             <geometry>
-                <box size="0.3 0.3 0.15"/>
+                <box size="${body_length} ${body_width} ${body_height}"/>
             </geometry>
             <material name="white"/>
         </visual>
         <collision>
-            <origin xyz="0.15 0 0.075"/>
+            <origin xyz="${body_mid_x} 0 ${body_mid_z}"/>
             <geometry>
-                <box size="0.3 0.3 0.15"/>
+                <box size="${body_length} ${body_width} ${body_height}"/>
             </geometry>
             <material name="white"/>
         </collision>
-        <xacro:inertial_box mass="0.5" x="0.3" y="0.3" z="0.15">
-            <origin xyz="0.15 0 0.075" rpy="0 0 0"/>
+        <xacro:inertial_box mass="${body_mass}" x="${body_length}" y="${body_width}" z="${body_height}">
+            <origin xyz="${body_mid_x} 0 ${body_mid_z}" rpy="0 0 0"/>
         </xacro:inertial_box>
     </link>
@@ -49,5 +72,5 @@
         <parent link="base_link"/>
         <child link="left_wheel_link"/>
-        <origin xyz="0 0.175 0" rpy="-${pi/2} 0 0"/>
+        <origin xyz="0 ${wheel_base_width} ${wheel_mount_height}" rpy="-${pi/2} 0 0"/>
         <axis xyz="0 0 1"/>
     </joint>
@@ -55,5 +78,5 @@
         <visual>
             <geometry>
-                <cylinder radius="0.05" length="0.04"/>
+                <cylinder radius="${drive_wheel_radius}" length="${drive_wheel_width}"/>
             </geometry>
             <material name="orange"/>
@@ -61,9 +84,9 @@
         <collision>
             <geometry>
-                <cylinder radius="0.05" length="0.04"/>
+                <cylinder radius="${drive_wheel_radius}" length="${drive_wheel_width}"/>
             </geometry>
             <material name="orange"/>
         </collision>
-        <xacro:inertial_cylinder mass="0.1" length="0.05" radius="0.05">
+        <xacro:inertial_cylinder mass="${drive_wheel_mass}" length="${drive_wheel_width}" radius="${drive_wheel_radius}">
             <origin xyz="0 0 0" rpy="0 0 0"/>
         </xacro:inertial_cylinder>
@@ -76,5 +99,5 @@
         <parent link="base_link"/>
         <child link="right_wheel_link"/>
-        <origin xyz="0 -0.175 0" rpy="${pi/2} 0 0"/>
+        <origin xyz="0 -${wheel_base_width} ${wheel_mount_height}" rpy="${pi/2} 0 0"/>
         <axis xyz="0 0 -1"/>
     </joint>
@@ -82,5 +105,5 @@
         <visual>
             <geometry>
-                <cylinder radius="0.05" length="0.04"/>
+                <cylinder radius="${drive_wheel_radius}" length="${drive_wheel_width}"/>
             </geometry>
             <material name="blue"/>
@@ -88,9 +111,9 @@
         <collision>
             <geometry>
-                <cylinder radius="0.05" length="0.04"/>
+                <cylinder radius="${drive_wheel_radius}" length="${drive_wheel_width}"/>
             </geometry>
             <material name="blue"/>
         </collision>
-        <xacro:inertial_cylinder mass="0.1" length="0.05" radius="0.05">
+        <xacro:inertial_cylinder mass="${drive_wheel_mass}" length="${drive_wheel_width}" radius="${drive_wheel_radius}">
             <origin xyz="0 0 0" rpy="0 0 0"/>
         </xacro:inertial_cylinder>
@@ -103,10 +126,10 @@
         <parent link="chassis_link"/>
         <child link="caster_wheel_link"/>
-        <origin xyz="0.24 0 0"/>
+        <origin xyz="${caster_x_pos} 0 0"/>
     </joint>
     <link name="caster_wheel_link">
         <visual>
             <geometry>
-                <sphere radius="0.05"/>
+                <sphere radius="${caster_radius}"/>
             </geometry>
             <material name="black"/>
@@ -114,9 +137,9 @@
         <collision>
             <geometry>
-                <sphere radius="0.05"/>
+                <sphere radius="${caster_radius}"/>
             </geometry>
             <material name="black"/>
         </collision>
-        <xacro:inertial_sphere mass="0.1" radius="0.05">
+        <xacro:inertial_sphere mass="${caster_mass}" radius="${caster_radius}">
             <origin xyz="0 0 0" rpy="0 0 0"/>
         </xacro:inertial_sphere>
@@ -124,7 +147,6 @@
     <gazebo reference="caster_wheel_link">
         <material>Gazebo/Black</material>
-        <!-- friction to reduce slipping -->
-        <mu1 value="0.001"/>
-        <mu2 value="0.001"/>
+        <mu1 value="${caster_friction_coeff}"/>
+        <mu2 value="${caster_friction_coeff}"/>
     </gazebo>
 </robot>

File: description/robot_core_real.xacro (robot description, xacro)
@@ -1,130 +1,148 @@
 <?xml version="1.0"?>
-<robot xmlns:xacro="http://www.ros.org/wiki/xacro" >
-    <xacro:include filename="inertial_macros.xacro" />
-    <material name="white">
-        <color rgba="1 1 1 1" />
-    </material>
-    <material name="blue">
-        <color rgba="0.2 0.2 1 1" />
-    </material>
-    <material name="orange">
-        <color rgba="1 0.3 0.1 1" />
-    </material>
-    <material name="black">
-        <color rgba="0 0 0 1" />
-    </material>
-    <!-- BASE LINK-->
-    <link name="base_link">
+<robot xmlns:xacro="http://www.ros.org/wiki/xacro" name="franky_bot">
+  <!-- =========================
+       Arguments (editable)
+       ========================= -->
+  <xacro:arg name="base_length"        default="0.34"/>
+  <xacro:arg name="base_width"         default="0.24"/>
+  <xacro:arg name="base_height"        default="0.14"/>
+  <xacro:arg name="wheel_radius"       default="0.034"/>
+  <xacro:arg name="wheel_width"        default="0.030"/>
+  <xacro:arg name="wheel_separation"   default="0.275"/>
+  <!-- Distances from edges -->
+  <xacro:arg name="d_front_wheel"      default="0.082"/>
+  <xacro:arg name="d_rear_caster"      default="0.065"/>
+  <xacro:arg name="caster_radius"      default="0.015"/>
+  <!-- =========================
+       Derived properties
+       ========================= -->
+  <xacro:property name="L" value="$(arg base_length)"/>
+  <xacro:property name="W" value="$(arg base_width)"/>
+  <xacro:property name="H" value="$(arg base_height)"/>
+  <xacro:property name="r_wheel" value="$(arg wheel_radius)"/>
+  <xacro:property name="w_wheel" value="$(arg wheel_width)"/>
+  <xacro:property name="b"       value="$(arg wheel_separation)"/>
+  <!-- Half-dimensions -->
+  <xacro:property name="L2" value="${L/2.0}"/>
+  <xacro:property name="W2" value="${W/2.0}"/>
+  <!-- Computed positions -->
+  <!-- wheel axle position from center: x = L/2 - d_front_wheel -->
+  <xacro:property name="x_wheel" value="${L2 - float($(arg d_front_wheel))}"/>
+  <!-- caster position from center: x = -(L/2 - d_rear_caster) -->
+  <xacro:property name="x_caster" value="${-(L2 - float($(arg d_rear_caster)))}"/>
+  <xacro:property name="y_left"  value="${ b/2.0}"/>
+  <xacro:property name="y_right" value="${-b/2.0}"/>
+  <xacro:property name="z_base"   value="${H/2.0}"/>
+  <xacro:property name="z_wheel"  value="${r_wheel}"/>
+  <xacro:property name="z_caster" value="${float($(arg caster_radius))}"/>
+  <!-- =========================
+       base_footprint (ground frame)
+       ========================= -->
+  <link name="base_footprint"/>
+  <joint name="base_footprint_to_base_link" type="fixed">
+    <parent link="base_footprint"/>
+    <child link="base_link"/>
+    <!-- base_link centered, lifted by half base height -->
+    <origin xyz="0 0 ${z_base}" rpy="0 0 0"/>
+  </joint>
+  <!-- =========================
+       base_link (main body)
+       ========================= -->
+  <link name="base_link">
+    <visual>
+      <origin xyz="0 0 0" rpy="0 0 0"/>
+      <geometry>
+        <box size="${L} ${W} ${H}"/>
+      </geometry>
+    </visual>
+    <collision>
+      <origin xyz="0 0 0" rpy="0 0 0"/>
+      <geometry>
+        <box size="${L} ${W} ${H}"/>
+      </geometry>
+    </collision>
+    <!-- Inertial: placeholder (tune later if you care about Gazebo physics) -->
+    <inertial>
+      <origin xyz="0 0 0" rpy="0 0 0"/>
+      <mass value="2.0"/>
+      <!-- rough inertia; replace with real values if needed -->
+      <inertia ixx="0.02" ixy="0.0" ixz="0.0"
+               iyy="0.03" iyz="0.0"
+               izz="0.04"/>
+    </inertial>
+  </link>
+  <!-- =========================
+       Wheel macro
+       ========================= -->
+  <xacro:macro name="wheel_link" params="name">
+    <link name="${name}">
+      <visual>
+        <!-- Cylinder axis is Z in URDF; rotate so it looks like a wheel (axis along Y) -->
+        <origin xyz="0 0 0" rpy="1.57079632679 0 0"/>
+        <geometry>
+          <cylinder radius="${r_wheel}" length="${w_wheel}"/>
+        </geometry>
+      </visual>
+      <collision>
+        <origin xyz="0 0 0" rpy="1.57079632679 0 0"/>
+        <geometry>
+          <cylinder radius="${r_wheel}" length="${w_wheel}"/>
+        </geometry>
+      </collision>
+      <inertial>
+        <origin xyz="0 0 0" rpy="0 0 0"/>
+        <mass value="0.2"/>
+        <inertia ixx="0.0002" ixy="0.0" ixz="0.0"
+                 iyy="0.0002" iyz="0.0"
+                 izz="0.0002"/>
+      </inertial>
     </link>
-    <!-- CHASSIS LINK-->
-    <joint name="chassis_joint" type="fixed">
-        <parent link="base_link" />
-        <child link="chassis_link" />
-        <origin xyz="-0.1 0 0"/>
-    </joint>
-    <link name="chassis_link">
-        <visual>
-            <origin xyz="0.15 0 0.075"/>
-            <geometry>
-                <box size="0.3 0.3 0.15"/>
-            </geometry>
-            <material name="white"/>
-        </visual>
-        <collision>
-            <origin xyz="0.15 0 0.075"/>
-            <geometry>
-                <box size="0.3 0.3 0.15"/>
-            </geometry>
-            <material name="white"/>
-        </collision>
-        <xacro:inertial_box mass="0.5" x="0.3" y="0.3" z="0.15">
-            <origin xyz="0.15 0 0.075" rpy="0 0 0"/>
-        </xacro:inertial_box>
-    </link>
-    <gazebo reference="chassis_link">
-        <material>Gazebo/Orange</material>
-    </gazebo>
-    <!-- LEFT WHEEL LINK-->
-    <joint name="left_wheel_joint" type="continuous">
-        <parent link="base_link"/>
-        <child link="left_wheel_link"/>
-        <origin xyz="0 0.175 0" rpy="-${pi/2} 0 0"/>
-        <axis xyz="0 0 1"/>
-    </joint>
-    <link name="left_wheel_link">
-        <visual>
-            <geometry>
-                <cylinder radius="0.05" length="0.04"/>
-            </geometry>
-            <material name="orange"/>
-        </visual>
-        <collision>
-            <geometry>
-                <cylinder radius="0.05" length="0.04"/>
-            </geometry>
-            <material name="orange"/>
-        </collision>
-        <xacro:inertial_cylinder mass="0.1" length="0.05" radius="0.05">
-            <origin xyz="0 0 0" rpy="0 0 0"/>
-        </xacro:inertial_cylinder>
-    </link>
-    <gazebo reference="left_wheel_link">
-        <material>Gazebo/Blue</material>
-    </gazebo>
-    <!-- RIGHT WHEEL LINK-->
-    <joint name="right_wheel_joint" type="continuous">
-        <parent link="base_link"/>
-        <child link="right_wheel_link"/>
-        <origin xyz="0 -0.175 0" rpy="${pi/2} 0 0"/>
-        <axis xyz="0 0 -1"/>
-    </joint>
-    <link name="right_wheel_link">
-        <visual>
-            <geometry>
-                <cylinder radius="0.05" length="0.04"/>
-            </geometry>
-            <material name="blue"/>
-        </visual>
-        <collision>
-            <geometry>
-                <cylinder radius="0.05" length="0.04"/>
-            </geometry>
-            <material name="blue"/>
-        </collision>
-        <xacro:inertial_cylinder mass="0.1" length="0.05" radius="0.05">
-            <origin xyz="0 0 0" rpy="0 0 0"/>
-        </xacro:inertial_cylinder>
-    </link>
-    <gazebo reference="right_wheel_link">
-        <material>Gazebo/Blue</material>
-    </gazebo>
-    <!-- CASTER WHEEL LINK-->
-    <joint name="caster_wheel_joint" type="fixed">
-        <parent link="chassis_link"/>
-        <child link="caster_wheel_link"/>
-        <origin xyz="0.24 0 0"/>
-    </joint>
-    <link name="caster_wheel_link">
-        <visual>
-            <geometry>
-                <sphere radius="0.05"/>
-            </geometry>
-            <material name="black"/>
-        </visual>
-        <collision>
-            <geometry>
-                <sphere radius="0.05"/>
-            </geometry>
-            <material name="black"/>
-        </collision>
-        <xacro:inertial_sphere mass="0.1" radius="0.05">
-            <origin xyz="0 0 0" rpy="0 0 0"/>
-        </xacro:inertial_sphere>
-    </link>
-    <gazebo reference="caster_wheel_link">
-        <material>Gazebo/Black</material>
-        <!-- friction to reduce slipping -->
-        <mu1 value="0.001"/>
-        <mu2 value="0.001"/>
-    </gazebo>
+  </xacro:macro>
+  <!-- Left wheel -->
+  <xacro:wheel_link name="left_wheel_link"/>
+  <joint name="left_wheel_joint" type="continuous">
+    <parent link="base_link"/>
+    <child link="left_wheel_link"/>
+    <origin xyz="${x_wheel} ${y_left} ${z_wheel}" rpy="0 0 0"/>
+    <!-- Wheel rotates around Y (left-right axis) -->
+    <axis xyz="0 1 0"/>
+  </joint>
+  <!-- Right wheel -->
+  <xacro:wheel_link name="right_wheel_link"/>
+  <joint name="right_wheel_joint" type="continuous">
+    <parent link="base_link"/>
+    <child link="right_wheel_link"/>
+    <origin xyz="${x_wheel} ${y_right} ${z_wheel}" rpy="0 0 0"/>
+    <axis xyz="0 1 0"/>
+  </joint>
+  <!-- =========================
+       Caster (simple visual)
+       ========================= -->
+  <link name="caster_link">
+    <visual>
+      <origin xyz="0 0 0" rpy="0 0 0"/>
+      <geometry>
+        <!-- Represent caster as sphere (good enough for RViz) -->
+        <sphere radius="$(arg caster_radius)"/>
+      </geometry>
+    </visual>
+    <collision>
+      <origin xyz="0 0 0" rpy="0 0 0"/>
+      <geometry>
+        <sphere radius="$(arg caster_radius)"/>
+      </geometry>
+    </collision>
+    <inertial>
+      <origin xyz="0 0 0" rpy="0 0 0"/>
+      <mass value="0.1"/>
+      <inertia ixx="0.00005" ixy="0.0" ixz="0.0"
+               iyy="0.00005" iyz="0.0"
+               izz="0.00005"/>
+    </inertial>
+  </link>
+  <joint name="caster_joint" type="fixed">
+    <parent link="base_link"/>
+    <child link="caster_link"/>
+    <origin xyz="${x_caster} 0 ${z_caster}" rpy="0 0 0"/>
+  </joint>
 </robot>

Commit message: ajustes en cámara

File: description/camera.xacro (robot description, xacro)
@@ -11,27 +11,23 @@
                 <box size="0.02 0.02 0.015"/>
             </geometry>
-            <!-- <material name="red"/> -->
+            <material name="black"/>
         </visual>
     </link>
+    <!-- No tiene forma, es solo para referenciar el frame optico de la camara, ajustando las coordenadas de ROS a las de Imagen -->
     <joint name="camera_optical_joint" type="fixed">
-        <origin xyz="0.01 0 0" rpy="${-pi/2} 0 ${-pi/2}" />
+        <origin xyz="0 0 0" rpy="${-pi/2} 0 ${-pi/2}" />
         <parent link="camera_link" />
         <child link="camera_optical_link" />
     </joint>
     <link name="camera_optical_link">
-        <visual>
-            <geometry>
-                <cylinder radius="0.004" length="0.002"/>
-            </geometry>
-            <!-- <material name="red"/> -->
-        </visual>
     </link>
     <gazebo reference="camera_link">
         <material>Gazebo/Red</material>
-        <sensor name="camera" type="camera">
+         <sensor name="camera" type="camera">
             <pose> 0 0 0 0 0 0 </pose>
             <visualize>true</visualize>
             <update_rate>10</update_rate>
             <camera>
+                <camera_info_topic>camera/camera_info</camera_info_topic>
                 <horizontal_fov>1.089</horizontal_fov>
                 <image>
@@ -45,5 +41,6 @@
                 </clip>
             </camera>
-            <topic>camera</topic>
+            <topic>camera/image_raw</topic>
+            <gz_frame_id>camera_link_optical</gz_frame_id>
         </sensor>
     </gazebo>
